File: projects/LTC7890_Buck/LTC7890_Buck.kicad_pcb (KiCad board)
At the start: 4 copper layers, 86 x 54 mm, 103 parts, among them J1 Bat In, J2 24V Out, J3 I2C Socket, J4 I2C Socket, Q1 IGC025S08S1, Q2 IGC025S08S1, Q3 IGC025S08S1, Q4 IGC025S08S1, SW1 Addr_Switch, SW2 Addr_Switch, U1 LTC7890, U2 TLV74033, U3 INA226

Commit message: Minor changes
Routing:
- net +3.3V: track 61.3 -> 61.6 mm, vias 2 -> 3
Changed lines of the file:
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@@
+		(net "+3.3V")
+	)
+	(via
+		(at 120 97.75)
+		(size 0.6)
+		(drill 0.3)
+		(layers "F.Cu" "B.Cu")
 		(net "+3.3V")
 	)
@@
 	)
 	(segment
-		(start 112.175 98.075)
+		(start 120 97.75)
+		(end 112.5 97.75)
+		(width 0.25)
+		(layer "In1.Cu")
+		(net "+3.3V")
+	)
+	(segment
+		(start 112.5 97.75)
 		(end 110.25 100)
 		(width 0.25)
@@
 	)
 	(segment
-		(start 143.4 98.075)
-		(end 112.175 98.075)
-		(width 0.25)
-		(layer "In1.Cu")
+		(start 146.925 98.075)
+		(end 143.4 98.075)
+		(width 0.25)
+		(layer "In2.Cu")
+		(net "+3.3V")
+	)
+	(segment
+		(start 134 97.75)
+		(end 143.075 97.75)
+		(width 0.25)
+		(layer "In2.Cu")
 		(net "+3.3V")
 	)
 	(segment
 		(start 152.75 97.25)
-		(end 151.925 98.075)
-		(width 0.25)
-		(layer "In2.Cu")
-		(net "+3.3V")
-	)
-	(segment
-		(start 151.925 98.075)
+		(end 147.75 97.25)
+		(width 0.25)
+		(layer "In2.Cu")
+		(net "+3.3V")
+	)
+	(segment
+		(start 134 97.75)
+		(end 120 97.75)
+		(width 0.25)
+		(layer "In2.Cu")
+		(net "+3.3V")
+	)
+	(segment
+		(start 147.75 97.25)
+		(end 146.925 98.075)
+		(width 0.25)
+		(layer "In2.Cu")
+		(net "+3.3V")
+	)
+	(segment
+		(start 143.075 97.75)
 		(end 143.4 98.075)
 		(width 0.25)
@@
 	)
 	(segment
+		(start 147.75 96.5)
+		(end 147 97.25)
+		(width 0.25)
+		(layer "In2.Cu")
+		(net "Net-(J3-Pin_3)")
+	)
+	(segment
 		(start 154.75 97.75)
 		(end 155.83704 97.75)
@@
 	)
 	(segment
+		(start 146.125 97.25)
+		(end 145.875 97)
+		(width 0.25)
+		(layer "In2.Cu")
+		(net "Net-(J3-Pin_3)")
+	)
+	(segment
+		(start 145.875 97)
+		(end 119.25 97)
+		(width 0.25)
+		(layer "In2.Cu")
+		(net "Net-(J3-Pin_3)")
+	)
+	(segment
+		(start 119.25 97)
+		(end 116.25 100)
+		(width 0.25)
+		(layer "In2.Cu")
+		(net "Net-(J3-Pin_3)")
+	)
+	(segment
 		(start 154.75 97.75)
 		(end 154.25 97.75)
@@
 	)
 	(segment
-		(start 147.25 97.25)
-		(end 119 97.25)
+		(start 153 96.5)
+		(end 147.75 96.5)
+		(width 0.25)
+		(layer "In2.Cu")
+		(net "Net-(J3-Pin_3)")
+	)
+	(segment
+		(start 156.33704 98.25)
+		(end 168 98.25)
 		(width 0.25)
 		(layer "In2.Cu")
@@
 	)
 	(segment
-		(start 156.33704 98.25)
-		(end 168 98.25)
-		(width 0.25)
-		(layer "In2.Cu")
-		(net "Net-(J3-Pin_3)")
-	)
-	(segment
-		(start 119 97.25)
-		(end 116.25 100)
-		(width 0.25)
-		(layer "In2.Cu")
-		(net "Net-(J3-Pin_3)")
-	)
-	(segment
-		(start 153 96.5)
-		(end 148 96.5)
-		(width 0.25)
-		(layer "In2.Cu")
-		(net "Net-(J3-Pin_3)")
-	)
-	(segment
-		(start 148 96.5)
-		(end 147.25 97.25)
+		(start 147 97.25)
+		(end 146.125 97.25)
 		(width 0.25)
 		(layer "In2.Cu")
@@
 	)
 	(segment
-		(start 146.25 96.5)
-		(end 142.25 100.5)
-		(width 0.25)
-		(layer "In1.Cu")
-		(net "/~{Alert}")
-	)
-	(segment
-		(start 146.5 96.5)
-		(end 146.25 96.5)
-		(width 0.25)
-		(layer "In1.Cu")
-		(net "/~{Alert}")
-	)
-	(segment
-		(start 142.25 100.5)
-		(end 139.75 100.5)
-		(width 0.25)
-		(layer "In1.Cu")
-		(net "/~{Alert}")
-	)
-	(segment
 		(start 139.75 100.5)
 		(end 139 101.25)
 		(width 0.25)
 		(layer "In1.Cu")
+		(net "/~{Alert}")
+	)
+	(segment
+		(start 142.5 100.5)
+		(end 139.75 100.5)
+		(width 0.25)
+		(layer "In1.Cu")
+		(net "/~{Alert}")
+	)
+	(segment
+		(start 146.5 96.5)
+		(end 142.5 100.5)
+		(width 0.25)
+		(layer "In1.Cu")

Commit message: New Revision
Parts:
- removed TP3, TP4: TestPoint, TestPoint:TestPoint_Keystone_5000-5004_Miniature
- removed TP5: TestPoint, TestPoint:TestPoint_Pad_D2.0mm
- added C32: 100nF, Capacitor_SMD:C_0603_1608Metric, B.Cu at (122.8, 97.8)
- added C33: 100nF, Capacitor_SMD:C_0603_1608Metric, B.Cu at (131.2, 97.8)
- added G***: LOGO, LOGO, B.Cu at (111.2, 133.0)
- added H1: MountingHole, MountingHole:MountingHole_3.2mm_M3, F.Cu at (101.0, 98.0)
- added H2: MountingHole, MountingHole:MountingHole_3.2mm_M3, F.Cu at (172.5, 93.0)
- added H3: MountingHole, MountingHole:MountingHole_3.2mm_M3, F.Cu at (100.5, 133.5)
- added H4: MountingHole, MountingHole:MountingHole_3.2mm_M3, F.Cu at (179.5, 133.5)
- added Q5: GSF3400, Package_TO_SOT_SMD:SOT-23, B.Cu at (121.0, 103.0)
- added R38: 8.2k, Resistor_SMD:R_0603_1608Metric, B.Cu at (150.8, 96.5)
- added R5: 10k, Resistor_SMD:R_0603_1608Metric, B.Cu at (125.8, 95.0)
- added R6: 10k, Resistor_SMD:R_0603_1608Metric, B.Cu at (117.8, 101.5)
- added SW3: SW_SP3T, footprints:CL-SB-13A, B.Cu at (162.5, 94.8)
- added SW4: SW_SP3T, footprints:CL-SB-13A, B.Cu at (117.5, 94.2)
- added TH1: JSNB103F344FBEWH, Resistor_SMD:R_0603_1608Metric, F.Cu at (140.0, 116.2)
- added U2: ADC101C021CIMM, Package_SO:MSOP-8_3x3mm_P0.65mm, B.Cu at (127.0, 97.8)
- SW1, SW2: value Addr_Switch -> SW_SP4T
- TP1, TP2: footprint TestPoint:TestPoint_Keystone_5000-5004_Miniature -> TestPoint:TestPoint_THTPad_D2.0mm_Drill1.0mm
- moved TP1 71.6 mm to (150.0, 135.2)
- moved TP2 51.4 mm to (130.0, 135.2)
- moved J3 11.9 mm to (177.8, 86.5), turned to 180 degrees
- moved J4 7.50 mm to (179.5, 95.8)
- moved C12 6.75 mm to (118.2, 90.2)
- moved C13 6.75 mm to (132.0, 90.2)
- moved C14 6.75 mm to (145.8, 90.2)
- moved C15 6.75 mm to (159.5, 90.2)
- moved J1 3.50 mm to (105.5, 85.0)
- moved L1 1.25 mm to (183.2, 116.0)
- moved L2 1.25 mm to (96.8, 116.0)
- moved D2 1.15 mm to (125.0, 114.8)
- moved D1 1.00 mm to (155.0, 115.0)
- moved SW1 0.50 mm to (113.2, 98.0)
- moved SW2 0.50 mm to (166.8, 98.0)
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- renumbered C32 to C34, C33 to C35, C34 to C36, C35 to C37, C36 to C38, C37 to C39, C38 to C40, C39 to C41, C40 to C42, C41 to C43, C42 to C44, C43 to C45, C44 to C46, R8 to R10, R9 to R11, R10 to R12, R11 to R13, R12 to R14, R13 to R15, R14 to R16, R15 to R17, R16 to R18, R17 to R19, R18 to R20, R19 to R21, R20 to R22, R21 to R23, R22 to R24, R23 to R25, R24 to R26, R25 to R27, R26 to R28, R27 to R29, R28 to R30, R29 to R31, R30 to R32, R31 to R33, R32 to R34, R33 to R35, R34 to R36, R35 to R37, R5 to R7, R6 to R8, R7 to R9, U2 to U3, U3 to U4
Connections:
- net Net-(J3-Pin_3) renamed /SDA
- net Net-(J3-Pin_4) renamed /SCL
- J1 pad 1: GNDPWR -> VDD
- J1 pad 2: VDD -> GNDPWR
- TP1 pad 1: VDD -> VOUT
- TP2 pad 1: GNDPWR -> Net-(Q5-D)
- U1 pad 17: Net-(D3-A) -> unconnected-(U1-PGOOD2-Pad17)
- U1 pad 34: unconnected-(U1-PGOOD1-Pad34) -> Net-(D3-A)
- U4 pad 3: /~{Alert} -> Net-(U4-~{Alert})
Routing:
- net +3.3V: track 61.6 -> 140.0 mm, vias 3 -> 9
- net Net-(U2-VIN): track 0.00 -> 59.3 mm, vias 0 -> 4
- net Net-(Q5-D): track 0.00 -> 42.3 mm, vias 0 -> 1
- net Net-(U2-ADR0): track 0.00 -> 36.7 mm, vias 0 -> 2
- net Net-(D3-A): track 4.59 -> 33.7 mm, vias 1 -> 2
- net GNDA: track 88.2 -> 111.8 mm, vias 8 -> 10
- net VOUT: track 80.6 -> 96.8 mm
- net Net-(U2-ADR1): track 0.00 -> 14.3 mm, vias 0 -> 2
- net Net-(Q5-G): track 0.00 -> 10.1 mm, vias 0 -> 2
- net Net-(U4-~{Alert}): track 0.00 -> 2.23 mm
- net Net-(R26-Pad1): track 9.26 -> 10.3 mm
- net /~{Alert}: track 18.4 -> 19.3 mm, vias 2 -> 3
- net Net-(U4-A1): track 20.3 -> 19.7 mm, vias 0 -> 1
- net /SCL: track 84.2 -> 83.6 mm
- net GNDPWR: vias 232 -> 224
Other:
- board text added: "24V Multiphase Buck Rev. 3 (40A Cont., 60A Max) Michael Lam"
- board text added: "DNP"
- board text added: "FAN+"
- board text added: "FAN-"
- board text removed: "+24V"
- board text removed: "BAT"
- board text removed: "GND"
- board text removed: "~{Alert}"
