File: projects/LTC7890_Buck/LTC7890_Buck.kicad_pcb (KiCad board)
At the start: 4 copper layers, 86 x 54 mm, 115 parts, among them J1 Bat In, J2 24V Out, J3 I2C Socket, J4 I2C Socket, Q1 IGC025S08S1, Q2 IGC025S08S1, Q3 IGC025S08S1, Q4 IGC025S08S1, Q5 GSF3400, SW1 SW_SP4T, SW2 SW_SP4T, SW3 SW_SP3T, SW4 SW_SP3T, U1 LTC7890, U2 ADC101C021CIMM, U3 TLV74033, U4 INA226

Commit message: Minor changes
Parts:
- added D4: V3PM10, footprints:D_SMP_DO-220AA, B.Cu at (140.0, 134.0)
- Q5: value GSF3400 -> PJA3438
- moved D2 0.15 mm to (125.0, 115.0)
- turned R6 to 180 degrees
Connections:
- R6 pad 1: +3.3V -> Net-(Q5-G)
- R6 pad 2: Net-(Q5-G) -> +3.3V
Routing:
- net Net-(D4-A): track 42.3 -> 52.0 mm, vias 1 -> 2
- net VOUT: track 96.8 -> 99.5 mm, vias 6 -> 7
Other:
- board text added: "< OUTPUT"
- board text added: "INPUT"
- board text added: "OUTPUT >"

Commit message: Minor rewiring
Connections:
- SW3 pad 1: +3.3V -> unconnected-(SW3-Pad1)
- SW3 pad 2: unconnected-(SW3-Pad2) -> GNDA
- SW3 pad 4: GNDA -> +3.3V
- SW4 pad 1: +3.3V -> unconnected-(SW4-Pad1)
- SW4 pad 2: unconnected-(SW4-Pad2) -> GNDA
- SW4 pad 4: GNDA -> +3.3V
Routing:
- net GNDA: track 111.8 -> 100.1 mm, vias 10 -> 9
- net +3.3V: track 140.0 -> 142.8 mm, vias 9 -> 11
